Commit message: update

File: chair_dance_sim/urdf/chair_robot.urdf.xacro (robot description, xacro)
@@ -208,32 +208,29 @@
   <xacro:caster name="front_right" parent_leg="front_right"/>
   <!-- ══════════════════════════════════════════════════════════════════════
-       Gazebo Plugins
+       Gz Sim (Fortress) Plugins
        ══════════════════════════════════════════════════════════════════════ -->
   <gazebo>
-    <!-- Differential drive controller -->
-    <plugin filename="libgazebo_ros_diff_drive.so" name="diff_drive">
-      <ros>
-        <remapping>cmd_vel:=/cmd_vel</remapping>
-        <remapping>odom:=/odom</remapping>
-      </ros>
+    <!-- Differential drive controller (Gz Sim system plugin) -->
+    <plugin filename="gz-sim-diff-drive-system"
+            name="gz::sim::systems::DiffDrive">
       <left_joint>back_left_wheel_joint</left_joint>
       <right_joint>back_right_wheel_joint</right_joint>
       <wheel_separation>${track}</wheel_separation>
-      <wheel_diameter>${wheel_r * 2}</wheel_diameter>
-      <max_wheel_torque>10.0</max_wheel_torque>
-      <max_wheel_acceleration>2.0</max_wheel_acceleration>
-      <!-- Odometry -->
-      <publish_odom>true</publish_odom>
-      <publish_odom_tf>true</publish_odom_tf>
-      <publish_wheel_tf>true</publish_wheel_tf>
-      <odometry_frame>odom</odometry_frame>
-      <robot_base_frame>base_footprint</robot_base_frame>
-      <update_rate>50.0</update_rate>
+      <wheel_radius>${wheel_r}</wheel_radius>
+      <max_linear_acceleration>2.0</max_linear_acceleration>
+      <odom_publish_frequency>50</odom_publish_frequency>
+      <topic>cmd_vel</topic>
+      <odom_topic>odom</odom_topic>
+      <tf_topic>tf</tf_topic>
+      <frame_id>odom</frame_id>
+      <child_frame_id>base_footprint</child_frame_id>
     </plugin>
     <!-- Joint state publisher for RViz -->
-    <plugin filename="libgazebo_ros_joint_state_publisher.so" name="joint_state_publisher">
+    <plugin filename="gz-sim-joint-state-publisher-system"
+            name="gz::sim::systems::JointStatePublisher">
       <joint_name>back_left_wheel_joint</joint_name>
       <joint_name>back_right_wheel_joint</joint_name>
       <update_rate>50</update_rate>
+      <topic>joint_states</topic>
     </plugin>
   </gazebo>
@@ -242,10 +239,8 @@
     <mu1>1.5</mu1>
     <mu2>1.5</mu2>
-    <material>Gazebo/DarkGrey</material>
   </gazebo>
   <gazebo reference="back_right_wheel">
     <mu1>1.5</mu1>
     <mu2>1.5</mu2>
-    <material>Gazebo/DarkGrey</material>
   </gazebo>
   <!-- Low friction on casters -->
@@ -253,29 +248,8 @@
     <mu1>0.001</mu1>
     <mu2>0.001</mu2>
-    <material>Gazebo/Grey</material>
   </gazebo>
   <gazebo reference="front_right_caster">
     <mu1>0.001</mu1>
     <mu2>0.001</mu2>
-    <material>Gazebo/Grey</material>
-  </gazebo>
-  <!-- Chair body colors in Gazebo -->
-  <gazebo reference="seat">
-    <material>Gazebo/FlatBlack</material>
-  </gazebo>
-  <gazebo reference="backrest">
-    <material>Gazebo/FlatBlack</material>
-  </gazebo>
-  <gazebo reference="back_left_leg">
-    <material>Gazebo/FlatBlack</material>
-  </gazebo>
-  <gazebo reference="back_right_leg">
-    <material>Gazebo/FlatBlack</material>
-  </gazebo>
-  <gazebo reference="front_left_leg">
-    <material>Gazebo/FlatBlack</material>
-  </gazebo>
-  <gazebo reference="front_right_leg">
-    <material>Gazebo/FlatBlack</material>
   </gazebo>
 </robot>
